File: ledstrip_digital_main/LED Strip rev 2.sch (KiCad schematic (older format))
At the start: 0 parts

Commit message: a little rearrangement and working on led motherboard
Parts:
- added C?: 100n, symbol C
- added C? (x2): 10p, symbol C
- added P?: CONN_4, symbol CONN_4
- added U?: STM32F051K8U8, MODULE, symbol STM32F051-32QFN
- added X?: 8M, symbol CRYSTAL
Connections:
- net labels added: +3.3V, GND, OSC_IN, OSC_OUT, SWCLK, SWDAT
- wire segments 0 -> 8
Changed lines of the file:
@@
-EESchema Schematic File Version 2  date Thu 26 Dec 2013 06:07:39 PM EST
+EESchema Schematic File Version 2  date Sun 05 Jan 2014 06:13:05 AM EST
 LIBS:power
 LIBS:device
@@
 LIBS:contrib
 LIBS:valves
-EELAYER 43  0
+LIBS:custom
+LIBS:LED Strip rev 2-cache
+EELAYER 25  0
 EELAYER END
 $Descr A4 11700 8267
@@
 Sheet 1 1
 Title ""
-Date "26 dec 2013"
+Date "5 jan 2014"
 Rev ""
 Comp ""
@@
 Comment4 ""
 $EndDescr
+Text Label 3600 3450 0    60   ~ 0
+OSC_OUT
+Text Label 3600 3350 0    60   ~ 0
+OSC_IN
+Wire Wire Line
+	4100 3450 3500 3450
+Wire Wire Line
+	7700 3950 7100 3950
+Wire Wire Line
+	6000 3250 6650 3250
+Connection ~ 2350 3750
+Connection ~ 2950 3750
+Wire Wire Line
+	2950 3150 2950 3750
+Wire Wire Line
+	2350 3750 2350 3200
+Wire Wire Line
+	6650 3350 6000 3350
+Wire Wire Line
+	7700 3750 7100 3750
+Wire Wire Line
+	4100 3350 3500 3350
+Text Label 2950 3600 1    60   ~ 0
+OSC_OUT
+Text Label 2350 3600 1    60   ~ 0
+OSC_IN
+Text Label 7200 3950 0    60   ~ 0
+SWDAT
+Text Label 7200 3750 0    60   ~ 0
+SWCLK
+$Comp
+L GND #PWR?
+U 1 1 52C93D8F
+P 7700 3850
+F 0 "#PWR?" H 7700 3850 30  0001 C CNN
+F 1 "GND" H 7700 3780 30  0001 C CNN
+	1    7700 3850
+	0    1    1    0
+$EndComp
+$Comp
+L +3.3V #PWR?
+U 1 1 52C93D8C
+P 7700 3650
+F 0 "#PWR?" H 7700 3610 30  0001 C CNN
+F 1 "+3.3V" H 7700 3760 30  0000 C CNN
+	1    7700 3650
+	0    -1   -1   0
+$EndComp
+$Comp
+L CONN_4 P?
+U 1 1 52C93D86
+P 8050 3800
+F 0 "P?" V 8000 3800 50  0000 C CNN
+F 1 "CONN_4" V 8100 3800 50  0000 C CNN
+	1    8050 3800
+	1    0    0    -1
+$EndComp
+Text Label 6200 3250 0    60   ~ 0
+SWCLK
+Text Label 6200 3350 0    60   ~ 0
+SWDAT
+$Comp
+L GND #PWR?
+U 1 1 52C93CB1
+P 2950 4150
+F 0 "#PWR?" H 2950 4150 30  0001 C CNN
+F 1 "GND" H 2950 4080 30  0001 C CNN
+	1    2950 4150
+	1    0    0    -1
+$EndComp
+$Comp
+L GND #PWR?
+U 1 1 52C93CAF
+P 2350 4150
+F 0 "#PWR?" H 2350 4150 30  0001 C CNN
+F 1 "GND" H 2350 4080 30  0001 C CNN
+	1    2350 4150
+	1    0    0    -1
+$EndComp
+$Comp
+L C C?
+U 1 1 52C93CA0
+P 2950 3950
+F 0 "C?" H 3000 4050 50  0000 L CNN
+F 1 "10p" H 3000 3850 50  0000 L CNN
+	1    2950 3950
+	1    0    0    -1
+$EndComp
+$Comp
+L C C?
+U 1 1 52C93C9C
+P 2350 3950
+F 0 "C?" H 2400 4050 50  0000 L CNN
+F 1 "10p" H 2400 3850 50  0000 L CNN
+	1    2350 3950
+	1    0    0    -1
+$EndComp
+$Comp
+L CRYSTAL X?
+U 1 1 52C93C96
+P 2650 3750
+F 0 "X?" H 2650 3900 60  0000 C CNN
+F 1 "8M" H 2650 3600 60  0000 C CNN
+	1    2650 3750
+	1    0    0    -1
+$EndComp
+$Comp
+L GND #PWR?
+U 1 1 52C93C8E
+P 4800 2650
+F 0 "#PWR?" H 4800 2650 30  0001 C CNN
+F 1 "GND" H 4800 2580 30  0001 C CNN
+	1    4800 2650
+	-1   0    0    1
+$EndComp
+$Comp
+L +3.3V #PWR?
+U 1 1 52C93C82
+P 3900 4100
+F 0 "#PWR?" H 3900 4060 30  0001 C CNN
+F 1 "+3.3V" H 3900 4210 30  0000 C CNN
+	1    3900 4100
+	1    0    0    -1
+$EndComp
+$Comp
+L GND #PWR?
+U 1 1 52C93C7F
+P 3900 4500
+F 0 "#PWR?" H 3900 4500 30  0001 C CNN
+F 1 "GND" H 3900 4430 30  0001 C CNN
+	1    3900 4500
+	1    0    0    -1
+$EndComp
+$Comp
+L C C?
+U 1 1 52C93C7C
+P 3900 4300
+F 0 "C?" H 3950 4400 50  0000 L CNN
+F 1 "100n" H 3950 4200 50  0000 L CNN
+	1    3900 4300
+	1    0    0    -1
+$EndComp
+$Comp
+L +3.3V #PWR?
+U 1 1 52C93C75
+P 6000 3950
+F 0 "#PWR?" H 6000 3910 30  0001 C CNN
+F 1 "+3.3V" H 6000 4060 30  0000 C CNN
+	1    6000 3950
+	0    1    1    0
+$EndComp
+$Comp
+L +3.3V #PWR?
+U 1 1 52C93C72
+P 4100 3650
+F 0 "#PWR?" H 4100 3610 30  0001 C CNN
+F 1 "+3.3V" H 4100 3760 30  0000 C CNN
+	1    4100 3650
+	0    -1   -1   0
+$EndComp
+$Comp
+L +3.3V #PWR?
+U 1 1 52C93C6E
+P 4100 3250
+F 0 "#PWR?" H 4100 3210 30  0001 C CNN
+F 1 "+3.3V" H 4100 3360 30  0000 C CNN
+	1    4100 3250
+	0    -1   -1   0
+$EndComp
+$Comp
+L GND #PWR?
+U 1 1 52C93C65
+P 5600 4550
+F 0 "#PWR?" H 5600 4550 30  0001 C CNN
+F 1 "GND" H 5600 4480 30  0001 C CNN
+	1    5600 4550
+	1    0    0    -1
+$EndComp
+$Comp
+L STM32F051-32QFN U?
+U 1 1 52C93C60
+P 5050 3600
+F 0 "U?" H 5050 3450 50  0000 C CNN
+F 1 "STM32F051K8U8" H 5050 3600 50  0000 C CNN
+F 2 "MODULE" H 5050 3600 50  0001 C CNN
+F 3 "DOCUMENTATION" H 5050 3600 50  0001 C CNN
+	1    5050 3600
+	1    0    0    -1
+$EndComp
 $EndSCHEMATC

Commit message: Schematic for digital LED motherboard basically done
Parts:
- added C? (x2): 100n, symbol C
- added C?: 10n, symbol C
- added P?: STRIP, symbol CONN_4
- added R? (x2): 0, symbol R
- added R? (x2): 1k, symbol R
- added R?: 15m, symbol R
- added R?: 470K, symbol R
- added R?: 100K, symbol R
- added R?: 1M, symbol R
- added U?: AURORA_CARD, MODULE, symbol AURORA_CARD
- added U?: TSC888B, symbol TSC888
- P?: value CONN_4 -> SWD
Connections:
- net labels added: +12V, +5V, I_LED, LED_CLK, LED_DAT, RTS, RX, TX, V_LED
- wire segments 8 -> 32
Other:
- moved on the sheet: C?, P?, U?, X?

Commit message: Finished up schematic for digital led motherboard
Parts:
- removed U?: AURORA_CARD, MODULE, symbol AURORA_CARD
- added C?: 1n, symbol C
- added CONN?: AURORA_CARD, MODULE, symbol AURORA_CARD
- C?: value 10n -> 1n
- R? (x2): value 1k -> 1K
- R?: value 470K -> 4.7M
- R?: value 100K -> 1M
Other:
- moved on the sheet: R?
Changed lines of the file:
@@
-EESchema Schematic File Version 2  date Sun 05 Jan 2014 08:35:43 AM EST
+EESchema Schematic File Version 2  date Sun 05 Jan 2014 08:48:54 AM EST
 LIBS:power
 LIBS:device
@@
 Comment4 ""
 $EndDescr
+Connection ~ 8400 1950
+Text Label 8550 1950 0    60   ~ 0
+V_LED
+Wire Wire Line
+	8150 1950 8900 1950
+Connection ~ 7350 2050
+Wire Wire Line
+	7350 2050 7800 2050
+Wire Wire Line
+	4300 4850 3700 4850
+Wire Wire Line
+	6800 3000 6800 3300
+Wire Wire Line
+	6800 3300 7250 3300
+Wire Wire Line
+	7850 3750 7850 3650
+Wire Wire Line
+	7850 3650 7750 3650
+Wire Wire Line
+	6200 4850 6850 4850
+Wire Wire Line
+	6200 4550 6850 4550
+Wire Wire Line
+	3850 3300 4350 3300
+Wire Wire Line
+	7850 3950 7250 3950
+Connection ~ 5500 3250
+Connection ~ 5300 3250
+Wire Wire Line
+	5500 3250 5500 2700
+Wire Wire Line
+	4300 4550 3700 4550
+Wire Wire Line
+	7900 5050 7300 5050
+Wire Wire Line
+	6200 4350 6850 4350
+Connection ~ 2550 4850
+Connection ~ 3150 4850
+Wire Wire Line
+	3150 4250 3150 4850
+Wire Wire Line
+	2550 4850 2550 4300
+Wire Wire Line
+	6850 4450 6200 4450
+Wire Wire Line
+	7900 4850 7300 4850
+Wire Wire Line
+	4300 4450 3700 4450
+Wire Wire Line
+	5300 3250 5300 2700
+Wire Wire Line
+	7850 3850 7250 3850
+Wire Wire Line
+	3850 3400 4350 3400
+Wire Wire Line
+	3850 3200 4350 3200
+Wire Wire Line
+	6200 4750 6850 4750
+Wire Wire Line
+	7250 3300 7250 3650
+Wire Wire Line
+	7750 3650 7750 3300
+Connection ~ 7250 3650
+Connection ~ 7750 3650
+Wire Wire Line
+	8150 3000 8150 3300
+Wire Wire Line
+	8150 3300 7750 3300
+Connection ~ 8150 1950
+Wire Wire Line
+	4300 4950 3700 4950
+Wire Wire Line
+	6850 2050 6800 2050
+Wire Wire Line
+	6800 2050 6800 2800
+$Comp
+L GND #PWR?
+U 1 1 52C961E9
+P 8400 2350
+F 0 "#PWR?" H 8400 2350 30  0001 C CNN
+F 1 "GND" H 8400 2280 30  0001 C CNN
+	1    8400 2350
+	1    0    0    -1
+$EndComp
+$Comp
+L C C?
+U 1 1 52C961E7
+P 8400 2150
+F 0 "C?" H 8450 2250 50  0000 L CNN
+F 1 "1n" H 8450 2050 50  0000 L CNN
+	1    8400 2150
+	1    0    0    -1
+$EndComp
+$Comp
+L +5V #PWR?
+U 1 1 52C960F1
+P 1750 3200
+F 0 "#PWR?" H 1750 3290 20  0001 C CNN
+F 1 "+5V" H 1750 3300 30  0000 C CNN
+	1    1750 3200
+	0    -1   -1   0
+$EndComp
+$Comp
+L AURORA_CARD CONN?
+U 1 1 52C960DA
+P 2800 3150
+F 0 "CONN?" H 2800 3050 50  0000 C CNN
+F 1 "AURORA_CARD" H 2800 3250 50  0000 C CNN
+F 2 "MODULE" H 2800 3150 50  0001 C CNN
+F 3 "DOCUMENTATION" H 2800 3150 50  0001 C CNN
+	1    2800 3150
+	-1   0    0    1
+$EndComp
 Text Label 7450 2050 0    60   ~ 0
 I_LED
-Wire Wire Line
-	6800 2800 6800 2050
-Wire Wire Line
-	6800 2050 6850 2050
-Wire Wire Line
-	4300 4950 3700 4950
-Connection ~ 9050 3450
-Wire Wire Line
-	9050 3450 8600 3450
-Wire Wire Line
-	8150 3300 7750 3300
-Wire Wire Line
-	8150 3300 8150 3000
-Connection ~ 7750 3650
-Connection ~ 7250 3650
-Wire Wire Line
-	7750 3300 7750 3650
-Wire Wire Line
-	7250 3650 7250 3300
-Wire Wire Line
-	6200 4750 6850 4750
-Wire Wire Line
-	2150 2950 1650 2950
-Wire Wire Line
-	2150 2750 1650 2750
-Wire Wire Line
-	7850 3850 7250 3850
-Wire Wire Line
-	5300 3250 5300 2700
-Wire Wire Line
-	4300 4450 3700 4450
-Wire Wire Line
-	7900 4850 7300 4850
-Wire Wire Line
-	6850 4450 6200 4450
-Wire Wire Line
-	2550 4850 2550 4300
-Wire Wire Line
-	3150 4250 3150 4850
-Connection ~ 3150 4850
-Connection ~ 2550 4850
-Wire Wire Line
-	6200 4350 6850 4350
-Wire Wire Line
-	7900 5050 7300 5050
-Wire Wire Line
-	4300 4550 3700 4550
-Wire Wire Line
-	5500 3250 5500 2700
-Connection ~ 5300 3250
-Connection ~ 5500 3250
-Wire Wire Line
-	7850 3950 7250 3950
-Wire Wire Line
-	2150 2850 1650 2850
-Wire Wire Line
-	6200 4550 6850 4550
-Wire Wire Line
-	6200 4850 6850 4850
-Wire Wire Line
-	7750 3650 7850 3650
-Wire Wire Line
-	7850 3650 7850 3750
-Wire Wire Line
-	7250 3300 6800 3300
-Wire Wire Line
-	6800 3300 6800 3000
-Wire Wire Line
-	4300 4850 3700 4850
-Wire Wire Line
-	7350 2050 7800 2050
-Connection ~ 7350 2050
 $Comp
 L GND #PWR?
@@
 P 7350 2250
 F 0 "C?" H 7400 2350 50  0000 L CNN
-F 1 "10n" H 7400 2150 50  0000 L CNN
+F 1 "1n" H 7400 2150 50  0000 L CNN
 	1    7350 2250
 	1    0    0    -1
@@
 Text Label 3800 4850 0    60   ~ 0
 V_LED
-Text Label 8650 3450 0    60   ~ 0
-V_LED
 $Comp
 L GND #PWR?
 U 1 1 52C95D56
-P 9050 3950
-F 0 "#PWR?" H 9050 3950 30  0001 C CNN
-F 1 "GND" H 9050 3880 30  0001 C CNN
-	1    9050 3950
+P 8150 2450
+F 0 "#PWR?" H 8150 2450 30  0001 C CNN
+F 1 "GND" H 8150 2380 30  0001 C CNN
+	1    8150 2450
 	1    0    0    -1
 $EndComp
@@
 L R R?
 U 1 1 52C95D53
-P 9050 3700
-F 0 "R?" V 9130 3700 50  0000 C CNN
-F 1 "100K" V 9050 3700 50  0000 C CNN
-	1    9050 3700
+P 8150 2200
+F 0 "R?" V 8230 2200 50  0000 C CNN
+F 1 "1M" V 8150 2200 50  0000 C CNN
+	1    8150 2200
 	1    0    0    -1
 $EndComp
@@
 L R R?
 U 1 1 52C95D51
-P 9050 3200
-F 0 "R?" V 9130 3200 50  0000 C CNN
-F 1 "470K" V 9050 3200 50  0000 C CNN
-	1    9050 3200
+P 8150 1700
+F 0 "R?" V 8230 1700 50  0000 C CNN
+F 1 "4.7M" V 8150 1700 50  0000 C CNN
+	1    8150 1700
 	1    0    0    -1
 $EndComp
@@
 L +12V #PWR?
 U 1 1 52C95D39
-P 9050 2950
-F 0 "#PWR?" H 9050 2900 20  0001 C CNN
-F 1 "+12V" H 9050 3050 30  0000 C CNN
-	1    9050 2950
+P 8150 1450
+F 0 "#PWR?" H 8150 1400 20  0001 C CNN
+F 1 "+12V" H 8150 1550 30  0000 C CNN
+	1    8150 1450
 	1    0    0    -1
 $EndComp
@@
 Text Label 6450 4850 0    60   ~ 0
 TX
-Text Label 1750 2950 0    60   ~ 0
+Text Label 4250 3200 2    60   ~ 0
 RTS
-Text Label 1750 2850 0    60   ~ 0
+Text Label 4250 3300 2    60   ~ 0
 TX
-Text Label 1750 2750 0    60   ~ 0
+Text Label 4250 3400 2    60   ~ 0
 RX
 $Comp
 L GND #PWR?
-U 1 1 52C9547C
-P 4250 3350
-F 0 "#PWR?" H 4250 3350 30  0001 C CNN
-F 1 "GND" H 4250 3280 30  0001 C CNN
-	1    4250 3350
-	0    -1   -1   0
-$EndComp
-$Comp
-L GND #PWR?
 U 1 1 52C9547A
-P 4250 3250
-F 0 "#PWR?" H 4250 3250 30  0001 C CNN
-F 1 "GND" H 4250 3180 30  0001 C CNN
-	1    4250 3250
-	0    -1   -1   0
+P 1750 3500
+F 0 "#PWR?" H 1750 3500 30  0001 C CNN
+F 1 "GND" H 1750 3430 30  0001 C CNN
+	1    1750 3500
+	0    1    1    0
 $EndComp
 $Comp
 L GND #PWR?
 U 1 1 52C95477
-P 2150 2650
-F 0 "#PWR?" H 2150 2650 30  0001 C CNN
-F 1 "GND" H 2150 2580 30  0001 C CNN
-	1    2150 2650
-	0    1    1    0
+P 3850 3500
+F 0 "#PWR?" H 3850 3500 30  0001 C CNN
+F 1 "GND" H 3850 3430 30  0001 C CNN
+	1    3850 3500
+	0    -1   -1   0
 $EndComp
 $Comp
 L +3.3V #PWR?
 U 1 1 52C9545E
-P 4250 3150
-F 0 "#PWR?" H 4250 3110 30  0001 C CNN
-F 1 "+3.3V" H 4250 3260 30  0000 C CNN
-	1    4250 3150
-	0    1    1    0
+P 1750 3400
+F 0 "#PWR?" H 1750 3360 30  0001 C CNN
+F 1 "+3.3V" H 1750 3510 30  0000 C CNN
+	1    1750 3400
+	0    -1   -1   0
 $EndComp
 $Comp
@@
 L +5V #PWR?
 U 1 1 52C95432
-P 4250 3050
-F 0 "#PWR?" H 4250 3140 20  0001 C CNN
-F 1 "+5V" H 4250 3200 30  0000 C CNN
-	1    4250 3050
-	0    1    1    0
+P 1750 3300
+F 0 "#PWR?" H 1750 3390 20  0001 C CNN
+F 1 "+5V" H 1750 3450 30  0000 C CNN
+	1    1750 3300
+	0    -1   -1   0
 $EndComp
 $Comp
 L +12V #PWR?
 U 1 1 52C9542E
-P 4250 2950
-F 0 "#PWR?" H 4250 2900 20  0001 C CNN
-F 1 "+12V" H 4250 3050 30  0000 C CNN
-	1    4250 2950
-	0    1    1    0
+P 1750 2800
+F 0 "#PWR?" H 1750 2750 20  0001 C CNN
+F 1 "+12V" H 1750 2900 30  0000 C CNN
+	1    1750 2800
+	0    -1   -1   0
 $EndComp
 $Comp
 L +12V #PWR?
 U 1 1 52C9542D
-P 4250 2850
-F 0 "#PWR?" H 4250 2800 20  0001 C CNN
-F 1 "+12V" H 4250 3000 30  0000 C CNN
-	1    4250 2850
-	0    1    1    0
+P 1750 2900
+F 0 "#PWR?" H 1750 2850 20  0001 C CNN
+F 1 "+12V" H 1750 3050 30  0000 C CNN
+	1    1750 2900
+	0    -1   -1   0
 $EndComp
 $Comp
 L +12V #PWR?
 U 1 1 52C9542C
-P 4250 2750
-F 0 "#PWR?" H 4250 2700 20  0001 C CNN
-F 1 "+12V" H 4250 2850 30  0000 C CNN
-	1    4250 2750
-	0    1    1    0
+P 1750 3000
+F 0 "#PWR?" H 1750 2950 20  0001 C CNN
+F 1 "+12V" H 1750 3100 30  0000 C CNN
+	1    1750 3000
+	0    -1   -1   0
 $EndComp
 $Comp
 L +12V #PWR?
 U 1 1 52C95428
-P 4250 2650
-F 0 "#PWR?" H 4250 2600 20  0001 C CNN
-F 1 "+12V" H 4250 2800 30  0000 C CNN
-	1    4250 2650
-	0    1    1    0
+P 1750 3100
+F 0 "#PWR?" H 1750 3050 20  0001 C CNN
+F 1 "+12V" H 1750 3250 30  0000 C CNN
+	1    1750 3100
+	0    -1   -1   0
 $EndComp
 $Comp
 L GND #PWR?
 U 1 1 52C95421
-P 2150 3350
-F 0 "#PWR?" H 2150 3350 30  0001 C CNN
-F 1 "GND" H 2150 3280 30  0001 C CNN
-	1    2150 3350
-	0    1    1    0
+P 3850 2800
+F 0 "#PWR?" H 3850 2800 30  0001 C CNN
+F 1 "GND" H 3850 2730 30  0001 C CNN
+	1    3850 2800
+	0    -1   -1   0
 $EndComp
 $Comp
 L GND #PWR?
 U 1 1 52C9541F
-P 2150 3250
-F 0 "#PWR?" H 2150 3250 30  0001 C CNN
-F 1 "GND" H 2150 3180 30  0001 C CNN
-	1    2150 3250
-	0    1    1    0
+P 3850 2900
+F 0 "#PWR?" H 3850 2900 30  0001 C CNN
+F 1 "GND" H 3850 2830 30  0001 C CNN
+	1    3850 2900
+	0    -1   -1   0
 $EndComp
 $Comp
 L GND #PWR?
 U 1 1 52C9541C
-P 2150 3150
-F 0 "#PWR?" H 2150 3150 30  0001 C CNN
-F 1 "GND" H 2150 3080 30  0001 C CNN
-	1    2150 3150
-	0    1    1    0
+P 3850 3000
+F 0 "#PWR?" H 3850 3000 30  0001 C CNN
+F 1 "GND" H 3850 2930 30  0001 C CNN
+	1    3850 3000
+	0    -1   -1   0
 $EndComp
 $Comp
 L GND #PWR?
 U 1 1 52C9541A
-P 2150 3050
-F 0 "#PWR?" H 2150 3050 30  0001 C CNN
-F 1 "GND" H 2150 2980 30  0001 C CNN
-	1    2150 3050
-	0    1    1    0
-$EndComp
-$Comp
-L AURORA_CARD U?
-U 1 1 52C9540D
-P 3200 3000
-F 0 "U?" H 3200 2900 50  0000 C CNN
-F 1 "AURORA_CARD" H 3200 3100 50  0000 C CNN
-F 2 "MODULE" H 3200 3000 50  0001 C CNN
-F 3 "DOCUMENTATION" H 3200 3000 50  0001 C CNN
-	1    3200 3000
-	1    0    0    -1
+P 3850 3100
+F 0 "#PWR?" H 3850 3100 30  0001 C CNN
+F 1 "GND" H 3850 3030 30  0001 C CNN
+	1    3850 3100
+	0    -1   -1   0
 $EndComp
 Text Label 7350 3950 0    60   ~ 0
@@
 P 5750 3250
 F 0 "R?" V 5830 3250 50  0000 C CNN
-F 1 "1k" V 5750 3250 50  0000 C CNN
+F 1 "1K" V 5750 3250 50  0000 C CNN
 	1    5750 3250
 	0    -1   -1   0
@@
 P 5050 3250
 F 0 "R?" V 5130 3250 50  0000 C CNN
-F 1 "1k" V 5050 3250 50  0000 C CNN
+F 1 "1K" V 5050 3250 50  0000 C CNN
 	1    5050 3250
 	0    1    1    0

Commit message: woo schematic
Parts:
- added D1: PWR, symbol LED
- added D2: USR, symbol LED
- added R1, R5: 1K, symbol R
- added R7, R8: R, symbol R
- added SW1: SW_PUSH, symbol SW_PUSH
- R10: renamed from R?; value 15m -> 10m
- R11: renamed from R?; value 4.7M -> 4M7
- gave numbers to parts that had none: 19
Connections:
- net labels added: USR_BTN, USR_LED
- wire segments 32 -> 36
- no-connect marks 0 -> 15
Other:
- moved on the sheet: C4

Commit message: worked on part placement, almost ready to begin routing
Parts:
- R7, R8: value R -> 330R
Changed lines of the file:
@@
 P 6700 5950
 F 0 "R8" V 6780 5950 50  0000 C CNN
-F 1 "R" V 6700 5950 50  0000 C CNN
+F 1 "330R" V 6700 5950 50  0000 C CNN
 F 2 "" H 6700 5950 60  0001 C CNN
 F 3 "" H 6700 5950 60  0001 C CNN
@@
 P 6250 5750
 F 0 "R7" V 6330 5750 50  0000 C CNN
-F 1 "R" V 6250 5750 50  0000 C CNN
+F 1 "330R" V 6250 5750 50  0000 C CNN
 F 2 "" H 6250 5750 60  0001 C CNN
 F 3 "" H 6250 5750 60  0001 C CNN
