File: ledstrip_digital_main/LED Strip rev 2.sch (KiCad schematic (older format))
At the start: 28 parts, among them P1 STRIP, P2 SWD, SW1 SW_PUSH, U1 STM32F051K8U8, U2 TSC888B, X1 8M

Commit message: finished copper for motherboard
Parts:
- removed SW1: SW_PUSH, symbol SW_PUSH
- added SW1: TACT, symbol TACT
Connections:
- net labels added: HP_GND
- wire segments 36 -> 44
Changed lines of the file:
@@
 Sheet 1 1
 Title ""
-Date "5 jan 2014"
+Date "6 jan 2014"
 Rev ""
 Comp ""
@@
 Comment4 ""
 $EndDescr
-Text Label 7100 5600 1    60   ~ 0
+Text Label 7250 5600 1    60   ~ 0
 USR_BTN
 Wire Wire Line
-	7100 5700 7100 5100
+	7250 5700 7250 5100
 Wire Wire Line
 	4900 5650 4900 6200
@@
 Connection ~ 5300 3250
 Wire Wire Line
-	5500 3250 5500 2450
+	5500 2450 5500 3250
 Wire Wire Line
 	4300 4550 3700 4550
@@
 	4300 4450 3700 4450
 Wire Wire Line
-	5300 3250 5300 2450
+	5300 2450 5300 3250
 Wire Wire Line
 	7850 3850 7250 3850
@@
 Connection ~ 8150 1950
 Wire Wire Line
-	4300 4950 3700 4950
-Wire Wire Line
 	6850 2050 6800 2050
 Wire Wire Line
@@
 L GND #PWR01
 U 1 1 52C96E16
-P 7100 6300
-F 0 "#PWR01" H 7100 6300 30  0001 C CNN
-F 1 "GND" H 7100 6230 30  0001 C CNN
-F 2 "" H 7100 6300 60  0001 C CNN
-F 3 "" H 7100 6300 60  0001 C CNN
-	1    7100 6300
-	1    0    0    -1
-$EndComp
-$Comp
-L SW_PUSH SW1
-U 1 1 52C96E08
-P 7100 6000
-F 0 "SW1" H 7250 6110 50  0000 C CNN
-F 1 "SW_PUSH" H 7100 5920 50  0000 C CNN
-F 2 "" H 7100 6000 60  0001 C CNN
-F 3 "" H 7100 6000 60  0001 C CNN
-	1    7100 6000
-	0    -1   -1   0
+P 7250 6600
+F 0 "#PWR01" H 7250 6600 30  0001 C CNN
+F 1 "GND" H 7250 6530 30  0001 C CNN
+F 2 "" H 7250 6600 60  0001 C CNN
+F 3 "" H 7250 6600 60  0001 C CNN
+	1    7250 6600
+	1    0    0    -1
 $EndComp
 Text Label 5000 6100 1    60   ~ 0
@@
 	0    1    1    0
 $EndComp
-Text Label 3800 4950 0    60   ~ 0
-I_LED
 Text Label 3800 4850 0    60   ~ 0
 V_LED
@@
 	0    -1   -1   0
 $EndComp
-$Comp
-L GND #PWR026
-U 1 1 52C95421
-P 3850 2800
-F 0 "#PWR026" H 3850 2800 30  0001 C CNN
-F 1 "GND" H 3850 2730 30  0001 C CNN
-F 2 "" H 3850 2800 60  0001 C CNN
-F 3 "" H 3850 2800 60  0001 C CNN
-	1    3850 2800
-	0    -1   -1   0
-$EndComp
-$Comp
-L GND #PWR027
-U 1 1 52C9541F
-P 3850 2900
-F 0 "#PWR027" H 3850 2900 30  0001 C CNN
-F 1 "GND" H 3850 2830 30  0001 C CNN
-F 2 "" H 3850 2900 60  0001 C CNN
-F 3 "" H 3850 2900 60  0001 C CNN
-	1    3850 2900
-	0    -1   -1   0
-$EndComp
-$Comp
-L GND #PWR028
-U 1 1 52C9541C
-P 3850 3000
-F 0 "#PWR028" H 3850 3000 30  0001 C CNN
-F 1 "GND" H 3850 2930 30  0001 C CNN
-F 2 "" H 3850 3000 60  0001 C CNN
-F 3 "" H 3850 3000 60  0001 C CNN
-	1    3850 3000
-	0    -1   -1   0
-$EndComp
-$Comp
-L GND #PWR029
-U 1 1 52C9541A
-P 3850 3100
-F 0 "#PWR029" H 3850 3100 30  0001 C CNN
-F 1 "GND" H 3850 3030 30  0001 C CNN
-F 2 "" H 3850 3100 60  0001 C CNN
-F 3 "" H 3850 3100 60  0001 C CNN
-	1    3850 3100
-	0    -1   -1   0
-$EndComp
 Text Label 7350 3950 0    60   ~ 0
 LED_CLK
@@
 LED_DAT
 $Comp
-L +12V #PWR030
+L +12V #PWR026
 U 1 1 52C951FD
 P 7250 3650
-F 0 "#PWR030" H 7250 3600 20  0001 C CNN
+F 0 "#PWR026" H 7250 3600 20  0001 C CNN
 F 1 "+12V" H 7250 3750 30  0000 C CNN
 F 2 "" H 7250 3650 60  0001 C CNN
@@
 	1    7250 3650
 	0    -1   -1   0
-$EndComp
-$Comp
-L GND #PWR031
-U 1 1 52C951F8
-P 7850 4050
-F 0 "#PWR031" H 7850 4050 30  0001 C CNN
-F 1 "GND" H 7850 3980 30  0001 C CNN
-F 2 "" H 7850 4050 60  0001 C CNN
-F 3 "" H 7850 4050 60  0001 C CNN
-	1    7850 4050
-	0    1    1    0
 $EndComp
 $Comp
@@
 LED_DAT
 $Comp
-L +5V #PWR032
+L +5V #PWR027
 U 1 1 52C950F3
 P 6000 3250
-F 0 "#PWR032" H 6000 3340 20  0001 C CNN
+F 0 "#PWR027" H 6000 3340 20  0001 C CNN
 F 1 "+5V" H 6000 3340 30  0000 C CNN
 F 2 "" H 6000 3250 60  0001 C CNN
@@
 $EndComp
 $Comp
-L +5V #PWR033
+L +5V #PWR028
 U 1 1 52C950ED
 P 4800 3250
-F 0 "#PWR033" H 4800 3340 20  0001 C CNN
+F 0 "#PWR028" H 4800 3340 20  0001 C CNN
 F 1 "+5V" H 4800 3340 30  0000 C CNN
 F 2 "" H 4800 3250 60  0001 C CNN
@@
 SWCLK
 $Comp
-L GND #PWR034
+L GND #PWR029
 U 1 1 52C93D8F
 P 7900 4950
-F 0 "#PWR034" H 7900 4950 30  0001 C CNN
+F 0 "#PWR029" H 7900 4950 30  0001 C CNN
 F 1 "GND" H 7900 4880 30  0001 C CNN
 F 2 "" H 7900 4950 60  0001 C CNN
@@
 $EndComp
 $Comp
-L +3.3V #PWR035
+L +3.3V #PWR030
 U 1 1 52C93D8C
 P 7900 4750
-F 0 "#PWR035" H 7900 4710 30  0001 C CNN
+F 0 "#PWR030" H 7900 4710 30  0001 C CNN
 F 1 "+3.3V" H 7900 4860 30  0000 C CNN
 F 2 "" H 7900 4750 60  0001 C CNN
@@
 SWDAT
 $Comp
-L GND #PWR036
+L GND #PWR031
 U 1 1 52C93CB1
 P 3150 5250
-F 0 "#PWR036" H 3150 5250 30  0001 C CNN
+F 0 "#PWR031" H 3150 5250 30  0001 C CNN
 F 1 "GND" H 3150 5180 30  0001 C CNN
 F 2 "" H 3150 5250 60  0001 C CNN
@@
 $EndComp
 $Comp
-L GND #PWR037
+L GND #PWR032
 U 1 1 52C93CAF
 P 2550 5250
-F 0 "#PWR037" H 2550 5250 30  0001 C CNN
+F 0 "#PWR032" H 2550 5250 30  0001 C CNN
 F 1 "GND" H 2550 5180 30  0001 C CNN
 F 2 "" H 2550 5250 60  0001 C CNN
@@
 $EndComp
 $Comp
-L GND #PWR038
+L GND #PWR033
 U 1 1 52C93C8E
 P 5000 3750
-F 0 "#PWR038" H 5000 3750 30  0001 C CNN
+F 0 "#PWR033" H 5000 3750 30  0001 C CNN
 F 1 "GND" H 5000 3680 30  0001 C CNN
 F 2 "" H 5000 3750 60  0001 C CNN
@@
 $EndComp
 $Comp
-L +3.3V #PWR039
+L +3.3V #PWR034
 U 1 1 52C93C82
 P 4100 5200
-F 0 "#PWR039" H 4100 5160 30  0001 C CNN
+F 0 "#PWR034" H 4100 5160 30  0001 C CNN
 F 1 "+3.3V" H 4100 5310 30  0000 C CNN
 F 2 "" H 4100 5200 60  0001 C CNN
@@
 $EndComp
 $Comp
-L GND #PWR040
+L GND #PWR035
 U 1 1 52C93C7F
 P 4100 5600
-F 0 "#PWR040" H 4100 5600 30  0001 C CNN
+F 0 "#PWR035" H 4100 5600 30  0001 C CNN
 F 1 "GND" H 4100 5530 30  0001 C CNN
 F 2 "" H 4100 5600 60  0001 C CNN
@@
 $EndComp
 $Comp
-L +3.3V #PWR041
+L +3.3V #PWR036
 U 1 1 52C93C75
 P 6200 5050
-F 0 "#PWR041" H 6200 5010 30  0001 C CNN
+F 0 "#PWR036" H 6200 5010 30  0001 C CNN
 F 1 "+3.3V" H 6200 5160 30  0000 C CNN
 F 2 "" H 6200 5050 60  0001 C CNN
@@
 $EndComp
 $Comp
-L +3.3V #PWR042
+L +3.3V #PWR037
 U 1 1 52C93C72
 P 4300 4750
-F 0 "#PWR042" H 4300 4710 30  0001 C CNN
+F 0 "#PWR037" H 4300 4710 30  0001 C CNN
 F 1 "+3.3V" H 4300 4860 30  0000 C CNN
 F 2 "" H 4300 4750 60  0001 C CNN
@@
 $EndComp
 $Comp
-L +3.3V #PWR043
+L +3.3V #PWR038
 U 1 1 52C93C6E
 P 4300 4350
-F 0 "#PWR043" H 4300 4310 30  0001 C CNN
+F 0 "#PWR038" H 4300 4310 30  0001 C CNN
 F 1 "+3.3V" H 4300 4460 30  0000 C CNN
 F 2 "" H 4300 4350 60  0001 C CNN
@@
 $EndComp
 $Comp
-L GND #PWR044
+L GND #PWR039
 U 1 1 52C93C65
 P 5800 5650
-F 0 "#PWR044" H 5800 5650 30  0001 C CNN
+F 0 "#PWR039" H 5800 5650 30  0001 C CNN
 F 1 "GND" H 5800 5580 30  0001 C CNN
 F 2 "" H 5800 5650 60  0001 C CNN
@@
 NoConn ~ 4300 5050
 NoConn ~ 5100 5650
-NoConn ~ 5200 5650
 NoConn ~ 5300 5650
 NoConn ~ 5400 5650
@@
 NoConn ~ 5400 3750
 NoConn ~ 5600 3750
+Wire Wire Line
+	7550 5700 7550 5800
+Wire Wire Line
+	7250 6500 7250 6600
+NoConn ~ 4300 4950
+Wire Wire Line
+	5200 5650 5200 6200
+Text Label 5200 6100 1    60   ~ 0
+I_LED
+Wire Wire Line
+	7850 4050 7250 4050
+Text Label 7350 4050 0    60   ~ 0
+HP_GND
+Wire Wire Line
+	3850 3100 3850 2800
+Wire Wire Line
+	3850 2800 4450 2800
+Text Label 3950 2800 0    60   ~ 0
+HP_GND
+Connection ~ 3850 2800
+Connection ~ 3850 2900
+Connection ~ 3850 3000
+$Comp
+L TACT SW1
+U 1 1 52CA51ED
+P 7250 6100
+F 0 "SW1" H 7250 6400 60  0000 C CNN
+F 1 "TACT" H 7250 5950 60  0000 C CNN
+F 2 "" H 7250 6100 60  0000 C CNN
+F 3 "" H 7250 6100 60  0000 C CNN
+	1    7250 6100
+	0    -1   -1   0
+$EndComp
+Wire Wire Line
+	7250 5700 7550 5700
+Wire Wire Line
+	7250 6500 6950 6500
+Wire Wire Line
+	6950 6500 6950 6400
 $EndSCHEMATC
