File: panelized/panelized.kicad_pcb (KiCad board)
At the start: 2 copper layers, 0 parts

Commit message: panelized
Parts:
- added C1: 2u2, SM1210, B.Cu at (179.5, 150.5)
- added C1: 10p, SM0402, F.Cu at (188.2, 132.5)
- added C1: 10p, SM0402, F.Cu at (157.2, 141.3)
- added C1: 47uF, SM1206, B.Cu at (185.2, 122.7)
- added C2: 2u2, SM0603, B.Cu at (188.0, 150.4)
- added C2: 10p, SM0402, F.Cu at (187.2, 132.5)
- added C2: 10p, SM0402, F.Cu at (158.2, 141.3)
- added C2: 1uF, SM0603_Capa, F.Cu at (156.0, 113.8)
- added C3: 1u, SM0603, B.Cu at (182.8, 150.4)
- added C3: 100n, SM0402, F.Cu at (182.5, 140.3)
- added C3: 100n, SM0402, F.Cu at (162.9, 133.5)
- added C3: 10uF, SM0805, B.Cu at (160.4, 120.1)
- added C4: 100n, SM0402, F.Cu at (180.6, 150.4)
- added C4: 100n, SM0402, F.Cu at (194.1, 136.4)
- added C4: 100n, SM0402, F.Cu at (151.3, 137.4)
- added C5: 5n6, SM0402, F.Cu at (179.1, 157.5)
- added C5: 1n, SM0402, F.Cu at (189.4, 136.0)
- added C5: 1n, SM0402, F.Cu at (156.0, 137.8)
- added C5: 100nF, SM0603_Capa, B.Cu at (160.4, 117.6)
- added C6: 120p, SM0402, F.Cu at (181.2, 157.5)
- added C6: 1n, SM0402, F.Cu at (186.2, 132.5)
- added C6: 1n, SM0402, F.Cu at (159.2, 141.3)
- added C6: 1uF, SM0603_Capa, B.Cu at (165.5, 119.5)
- added C7: 10u, SM1206, B.Cu at (191.2, 156.0)
- added C7: 100n, SM0402, F.Cu at (189.4, 135.0)
- added C7: 100n, SM0402, F.Cu at (156.0, 138.8)
- added C7: 1uF, SM0603_Capa, F.Cu at (161.1, 113.8)
- added C8: 10u, SM1206, B.Cu at (191.2, 158.4)
- added C8: 10uF, SM0805, F.Cu at (187.1, 122.7)
- added CONN1: AURORA_CARD, AURORA_CARD, F.Cu at (187.5, 154.2)
- added CONN1: AURORA_CARD, AURORA_CARD, F.Cu at (187.5, 136.9)
- added CONN1: AURORA_CARD, AURORA_CARD, F.Cu at (157.9, 136.9)
- added D1: 50WQ10FN, DPAK2, B.Cu at (186.7, 155.6)
- added D1: PWR, LED-0603, B.Cu at (175.4, 142.4)
- added D1: PWR, LED-0603, B.Cu at (170.0, 131.4)
- added D1: TX, LED-0603, F.Cu at (150.3, 125.6)
- added D2: USR, LED-0603, B.Cu at (175.4, 131.5)
- added D2: USR, LED-0603, B.Cu at (170.0, 142.4)
- added D2: RX, LED-0603, F.Cu at (150.3, 122.0)
- added D3: PWR, LED-0603, F.Cu at (150.3, 118.5)
- added D4: 12V, LED-0603, F.Cu at (150.3, 114.9)
- added GS1: GS3, S_JUMPER_3, F.Cu at (154.8, 119.2)
- added L1: 33u, MSS1210, F.Cu at (191.1, 154.2)
- added P1: Modular Jack In, Assman-6p4c, F.Cu at (165.9, 154.2)
- added P1: STRIP, SIL-4, F.Cu at (196.3, 136.9)
- added P1: STRIP, SIL-4, F.Cu at (149.0, 136.9)
- added P1: CONN_1, 1PIN_S_SMD, B.Cu at (161.7, 114.4)
- added P2: SWD, SMD-HDR-4, F.Cu at (180.5, 136.9)
- added P2: SWD, SMD-HDR-4, F.Cu at (164.9, 136.9)
- added P3: CONN_2, JACK_ALIM, F.Cu at (177.6, 118.2)
- added R1: 120R, SM1206, B.Cu at (172.9, 159.3)
- added R1: 1K, SM0402, F.Cu at (191.8, 139.5)
- added R1: 1K, SM0402, F.Cu at (153.6, 134.4)
- added R1: 270, SM0603, F.Cu at (150.3, 124.1)
- added R10: 10m, SM1206, F.Cu at (191.9, 133.1)
- added R10: 10m, SM1206, F.Cu at (153.5, 140.7)
- added R11: 4M7, SM0402, F.Cu at (184.2, 133.1)
- added R11: 4M7, SM0402, F.Cu at (161.2, 140.7)
- added R12: 1M, SM0402, F.Cu at (185.2, 132.5)
- added R12: 1M, SM0402, F.Cu at (160.2, 141.3)
- added R2: 221k, SM0402, F.Cu at (178.1, 157.5)
- added R2: 1K, SM0402, F.Cu at (192.8, 139.5)
- added R2: 1K, SM0402, F.Cu at (152.6, 134.4)
- added R2: 270, SM0603, F.Cu at (150.3, 120.5)
- added R3: 6K19, SM0402, F.Cu at (180.1, 157.5)
- added R3: 0, SM0402, F.Cu at (190.8, 139.5)
- added R3: 0, SM0402, F.Cu at (154.6, 134.4)
- added R3: 270, SM0603, F.Cu at (150.3, 117.0)
- added R4: 143k, SM0402, F.Cu at (183.2, 157.5)
- added R4: 0, SM0402, F.Cu at (190.8, 141.2)
- added R4: 0, SM0402, F.Cu at (154.6, 132.6)
- added R4: 10K, SM0603, F.Cu at (150.3, 113.4)
- added R5: 10k2, SM0402, F.Cu at (182.2, 157.5)
- added R5: 1K, SM0402, F.Cu at (191.8, 141.2)
- added R5: 1K, SM0402, F.Cu at (153.6, 132.6)
- added R6: 1K, SM0402, F.Cu at (192.8, 141.2)
- added R6: 1K, SM0402, F.Cu at (152.6, 132.6)
- added R7: 330R, SM0402, F.Cu at (182.5, 141.5)
- added R7: 330R, SM0402, F.Cu at (162.9, 132.3)
- added R8: 330R, SM0402, F.Cu at (182.1, 133.0)
- added R8: 330R, SM0402, F.Cu at (163.2, 140.8)
- added R9: 1M, SM0402, F.Cu at (189.4, 137.0)
- added R9: 1M, SM0402, F.Cu at (156.0, 136.8)
- added SW1: TACT, TACT-SW-SMD, B.Cu at (179.6, 136.9)
- added SW1: TACT, TACT-SW-SMD, B.Cu at (165.8, 136.9)
- added U1: LD1117, sot89, B.Cu at (192.3, 151.3)
- added U1: STM32F051K8U8, QFN32-5x5, F.Cu at (184.9, 136.9)
- added U1: STM32F051K8U8, QFN32-5x5, F.Cu at (160.5, 136.9)
- added U1: AURORA_CARD, AURORA_CARD, F.Cu at (178.2, 119.5)
- added U2: AP73333, SOT23, B.Cu at (185.3, 150.4)
- added U2: TSC888B, SOT23-5, F.Cu at (191.9, 136.3)
- added U2: TSC888B, SOT23-5, F.Cu at (153.5, 137.5)
- added U2: MICRO-B_USB, MICRO-B_USB, B.Cu at (148.0, 118.9)
- added U3: ST485E, SO8E, B.Cu at (167.2, 154.2)
- added U3: FT232RL, SSOP28, F.Cu at (160.4, 120.8)
- added U4: TPS54360DDAR, SO8_WITH_EP, F.Cu at (180.6, 153.7)
- added U4: AP7333, SOT23, F.Cu at (166.1, 114.4)
- added U5: LD1117, SOT223, B.Cu at (170.6, 119.5)
- added X1: 8M, CX5, B.Cu at (185.5, 136.9)
- added X1: 8M, CX5, B.Cu at (159.8, 136.9)
Routing:
- net GND: track 0.00 -> 225.7 mm, vias 0 -> 8
- net +12V: track 0.00 -> 165.6 mm, vias 0 -> 15
- net +5V: track 0.00 -> 101.2 mm, vias 0 -> 7
- net +3.3V: track 0.00 -> 62.0 mm, vias 0 -> 8
- net /OSC_OUT: track 0.00 -> 43.6 mm, vias 0 -> 2
- net /SWDAT: track 0.00 -> 34.0 mm, vias 0 -> 4
- net /SWCLK: track 0.00 -> 33.2 mm, vias 0 -> 4
- net /HP_GND: track 0.00 -> 32.6 mm
- net /RX: track 0.00 -> 27.0 mm, vias 0 -> 2
- net N-000004: track 0.00 -> 25.6 mm, vias 0 -> 1
- net /I_LED: track 0.00 -> 24.1 mm, vias 0 -> 4
- net N-000008: track 0.00 -> 22.9 mm, vias 0 -> 1
- net /RTS: track 0.00 -> 22.2 mm, vias 0 -> 1
- net N-000003: track 0.00 -> 18.5 mm, vias 0 -> 1
- net /TX: track 0.00 -> 18.2 mm
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- added copper zone on B.Cu, net +12V
- added copper zone on F.Cu, net +12V
- added copper zone on B.Cu, net +3.3V
- added copper zone on B.Cu, net GND
- added copper zone on F.Cu, net GND
Other:
- board outline added: 50 x 50 mm
- net class Default: clearance 0.254 -> 0.2032; trace_width 0.254 -> 0.2032
- rule trace_clearance: 0.254 -> 0.2032
- rule trace_min: 0.254 -> 0.1524
- rule via_min_drill: 0.508 -> 0.381
- rule via_min_size: 0.889 -> 0.762
- board text added: "+12V cpos"
- board text added: "1"
- board text added: "Aurora Project Digital LED Strip"
- board text added: "Aurora Project LUX Interface"
- board text added: "CLK"
- board text added: "DAT"
- board text added: "GND"
- board text added: "PWR"
- board text added: "aurora"
- board text added: "r1"
- board text added: "rev 1"
- board text added: "zbanks@mit.edu"
