File: lux_router_arm/out_port.sch (KiCad schematic (older format))
At the start: 7 parts

Commit message: Prelimary parts assignment to lux router
Parts:
- removed R?: R, symbol R
- added R13: 120, symbol R
- C13: renamed from C?; value C -> 100nF
- R14: renamed from R?; value R -> 1k
- gave numbers to parts that had none: 4
Connections:
- net at P8.2 (P2), U5.6 (A): now also R13.2
- net at P8.3 (P3), U5.7 (B): now also R13.1
Changed lines of the file:
@@
-EESchema Schematic File Version 2  date Thu 16 Jan 2014 03:35:13 AM EST
+EESchema Schematic File Version 2  date Thu 16 Jan 2014 04:47:59 AM EST
 LIBS:power
 LIBS:device
@@
 $Descr A4 11700 8267
 encoding utf-8
-Sheet 2 8
+Sheet 7 8
 Title ""
 Date "16 jan 2014"
@@
 Comment4 ""
 $EndDescr
+$Comp
+L R R13
+U 1 1 52D7A7A0
+P 6000 3900
+AR Path="/52D79664/52D7A7A0" Ref="R13"  Part="1"
+AR Path="/52D7966E/52D7A7A0" Ref="R7"  Part="1"
+AR Path="/52D7966D/52D7A7A0" Ref="R9"  Part="1"
+AR Path="/52D7966B/52D7A7A0" Ref="R11"  Part="1"
+AR Path="/52D79663/52D7A7A0" Ref="R15"  Part="1"
+AR Path="/52D7965C/52D7A7A0" Ref="R17"  Part="1"
+AR Path="/52D79548/52D7A7A0" Ref="R19"  Part="1"
+F 0 "R17" V 6080 3900 50  0000 C CNN
+F 1 "120" V 6000 3900 50  0000 C CNN
+	1    6000 3900
+	0    -1   -1   0
+$EndComp
 Wire Wire Line
 	4450 4700 4450 4800
@@
 	4450 5300 4450 5200
 $Comp
-L +5V #PWR?
+L +5V #PWR052
 U 1 1 52D7960C
 P 4450 4700
-F 0 "#PWR?" H 4450 4790 20  0001 C CNN
+AR Path="/52D79664/52D7960C" Ref="#PWR052"  Part="1"
+AR Path="/52D7966E/52D7960C" Ref="#PWR034"  Part="1"
+AR Path="/52D7966D/52D7960C" Ref="#PWR040"  Part="1"
+AR Path="/52D7966B/52D7960C" Ref="#PWR046"  Part="1"
+AR Path="/52D79663/52D7960C" Ref="#PWR058"  Part="1"
+AR Path="/52D7965C/52D7960C" Ref="#PWR064"  Part="1"
+AR Path="/52D79548/52D7960C" Ref="#PWR070"  Part="1"
+F 0 "#PWR064" H 4450 4790 20  0001 C CNN
 F 1 "+5V" H 4450 4790 30  0000 C CNN
 	1    4450 4700
@@
 $EndComp
 $Comp
-L GND #PWR?
+L GND #PWR053
 U 1 1 52D79608
 P 4450 5300
-F 0 "#PWR?" H 4450 5300 30  0001 C CNN
+AR Path="/52D79664/52D79608" Ref="#PWR053"  Part="1"
+AR Path="/52D7966E/52D79608" Ref="#PWR035"  Part="1"
+AR Path="/52D7966D/52D79608" Ref="#PWR041"  Part="1"
+AR Path="/52D7966B/52D79608" Ref="#PWR047"  Part="1"
+AR Path="/52D79663/52D79608" Ref="#PWR059"  Part="1"
+AR Path="/52D7965C/52D79608" Ref="#PWR065"  Part="1"
+AR Path="/52D79548/52D79608" Ref="#PWR071"  Part="1"
+F 0 "#PWR065" H 4450 5300 30  0001 C CNN
 F 1 "GND" H 4450 5230 30  0001 C CNN
 	1    4450 5300
@@
 $EndComp
 $Comp
-L GND #PWR?
+L GND #PWR054
 U 1 1 52D79605
 P 3650 5300
-F 0 "#PWR?" H 3650 5300 30  0001 C CNN
+AR Path="/52D79664/52D79605" Ref="#PWR054"  Part="1"
+AR Path="/52D7966E/52D79605" Ref="#PWR036"  Part="1"
+AR Path="/52D7966D/52D79605" Ref="#PWR042"  Part="1"
+AR Path="/52D7966B/52D79605" Ref="#PWR048"  Part="1"
+AR Path="/52D79663/52D79605" Ref="#PWR060"  Part="1"
+AR Path="/52D7965C/52D79605" Ref="#PWR066"  Part="1"
+AR Path="/52D79548/52D79605" Ref="#PWR072"  Part="1"
+F 0 "#PWR066" H 3650 5300 30  0001 C CNN
 F 1 "GND" H 3650 5230 30  0001 C CNN
 	1    3650 5300
@@
 TX
 $Comp
-L +5V #PWR?
+L +5V #PWR055
 U 1 1 52D795DE
 P 5300 3550
-F 0 "#PWR?" H 5300 3640 20  0001 C CNN
+AR Path="/52D79664/52D795DE" Ref="#PWR055"  Part="1"
+AR Path="/52D7966E/52D795DE" Ref="#PWR037"  Part="1"
+AR Path="/52D7966D/52D795DE" Ref="#PWR043"  Part="1"
+AR Path="/52D7966B/52D795DE" Ref="#PWR049"  Part="1"
+AR Path="/52D79663/52D795DE" Ref="#PWR061"  Part="1"
+AR Path="/52D7965C/52D795DE" Ref="#PWR067"  Part="1"
+AR Path="/52D79548/52D795DE" Ref="#PWR073"  Part="1"
+F 0 "#PWR067" H 5300 3640 20  0001 C CNN
 F 1 "+5V" H 5300 3640 30  0000 C CNN
 	1    5300 3550
@@
 $EndComp
 $Comp
-L +48V #PWR?
+L +48V #PWR056
 U 1 1 52D795D8
 P 6550 3000
-F 0 "#PWR?" H 6550 3130 20  0001 C CNN
+AR Path="/52D79664/52D795D8" Ref="#PWR056"  Part="1"
+AR Path="/52D7966E/52D795D8" Ref="#PWR038"  Part="1"
+AR Path="/52D7966D/52D795D8" Ref="#PWR044"  Part="1"
+AR Path="/52D7966B/52D795D8" Ref="#PWR050"  Part="1"
+AR Path="/52D79663/52D795D8" Ref="#PWR062"  Part="1"
+AR Path="/52D7965C/52D795D8" Ref="#PWR068"  Part="1"
+AR Path="/52D79548/52D795D8" Ref="#PWR074"  Part="1"
+F 0 "#PWR068" H 6550 3130 20  0001 C CNN
 F 1 "+48V" H 6550 3100 30  0000 C CNN
 	1    6550 3000
@@
 $EndComp
 $Comp
-L GND #PWR?
+L GND #PWR057
 U 1 1 52D795D1
 P 6000 4300
-F 0 "#PWR?" H 6000 4300 30  0001 C CNN
+AR Path="/52D79664/52D795D1" Ref="#PWR057"  Part="1"
+AR Path="/52D7966E/52D795D1" Ref="#PWR039"  Part="1"
+AR Path="/52D7966D/52D795D1" Ref="#PWR045"  Part="1"
+AR Path="/52D7966B/52D795D1" Ref="#PWR051"  Part="1"
+AR Path="/52D79663/52D795D1" Ref="#PWR063"  Part="1"
+AR Path="/52D7965C/52D795D1" Ref="#PWR069"  Part="1"
+AR Path="/52D79548/52D795D1" Ref="#PWR075"  Part="1"
+F 0 "#PWR069" H 6000 4300 30  0001 C CNN
 F 1 "GND" H 6000 4230 30  0001 C CNN
 	1    6000 4300
@@
 $EndComp
 $Comp
-L R R?
-U 1 1 52D795BB
-P 6000 3900
-F 0 "R?" V 6080 3900 50  0000 C CNN
-F 1 "R" V 6000 3900 50  0000 C CNN
-	1    6000 3900
-	0    -1   -1   0
-$EndComp
-$Comp
-L FUSE F?
+L FUSE F4
 U 1 1 52D795B4
 P 6550 3350
-F 0 "F?" H 6650 3400 40  0000 C CNN
+AR Path="/52D79664/52D795B4" Ref="F4"  Part="1"
+AR Path="/52D7966E/52D795B4" Ref="F1"  Part="1"
+AR Path="/52D7966D/52D795B4" Ref="F2"  Part="1"
+AR Path="/52D7966B/52D795B4" Ref="F3"  Part="1"
+AR Path="/52D79663/52D795B4" Ref="F5"  Part="1"
+AR Path="/52D7965C/52D795B4" Ref="F6"  Part="1"
+AR Path="/52D79548/52D795B4" Ref="F7"  Part="1"
+F 0 "F6" H 6650 3400 40  0000 C CNN
 F 1 "FUSE" H 6450 3300 40  0000 C CNN
 	1    6550 3350
@@
 $EndComp
 $Comp
-L C C?
+L C C13
 U 1 1 52D795AC
 P 4450 5000
-F 0 "C?" H 4500 5100 50  0000 L CNN
-F 1 "C" H 4500 4900 50  0000 L CNN
+AR Path="/52D79664/52D795AC" Ref="C13"  Part="1"
+AR Path="/52D7966E/52D795AC" Ref="C10"  Part="1"
+AR Path="/52D7966D/52D795AC" Ref="C11"  Part="1"
+AR Path="/52D7966B/52D795AC" Ref="C12"  Part="1"
+AR Path="/52D79663/52D795AC" Ref="C14"  Part="1"
+AR Path="/52D7965C/52D795AC" Ref="C15"  Part="1"
+AR Path="/52D79548/52D795AC" Ref="C16"  Part="1"
+F 0 "C15" H 4500 5100 50  0000 L CNN
+F 1 "100nF" H 4500 4900 50  0000 L CNN
 	1    4450 5000
 	1    0    0    -1
 $EndComp
 $Comp
-L R R?
+L R R14
 U 1 1 52D795AA
 P 3650 4450
-F 0 "R?" V 3730 4450 50  0000 C CNN
-F 1 "R" V 3650 4450 50  0000 C CNN
+AR Path="/52D79664/52D795AA" Ref="R14"  Part="1"
+AR Path="/52D7966E/52D795AA" Ref="R8"  Part="1"
+AR Path="/52D7966D/52D795AA" Ref="R10"  Part="1"
+AR Path="/52D7966B/52D795AA" Ref="R12"  Part="1"
+AR Path="/52D79663/52D795AA" Ref="R16"  Part="1"
+AR Path="/52D7965C/52D795AA" Ref="R18"  Part="1"
+AR Path="/52D79548/52D795AA" Ref="R20"  Part="1"
+F 0 "R18" V 3730 4450 50  0000 C CNN
+F 1 "1k" V 3650 4450 50  0000 C CNN
 	1    3650 4450
 	1    0    0    -1
 $EndComp
 $Comp
-L LED D?
+L LED D9
 U 1 1 52D795A3
 P 3650 5000
-F 0 "D?" H 3650 5100 50  0000 C CNN
+AR Path="/52D79664/52D795A3" Ref="D9"  Part="1"
+AR Path="/52D7966E/52D795A3" Ref="D6"  Part="1"
+AR Path="/52D7966D/52D795A3" Ref="D7"  Part="1"
+AR Path="/52D7966B/52D795A3" Ref="D8"  Part="1"
+AR Path="/52D79663/52D795A3" Ref="D10"  Part="1"
+AR Path="/52D7965C/52D795A3" Ref="D11"  Part="1"
+AR Path="/52D79548/52D795A3" Ref="D12"  Part="1"
+F 0 "D11" H 3650 5100 50  0000 C CNN
 F 1 "LED" H 3650 4900 50  0000 C CNN
 	1    3650 5000
@@
 $EndComp
 $Comp
-L CONN_4 P?
+L CONN_4 P8
 U 1 1 52D79591
 P 7050 3900
-F 0 "P?" V 7000 3900 50  0000 C CNN
+AR Path="/52D79664/52D79591" Ref="P8"  Part="1"
+AR Path="/52D7966E/52D79591" Ref="P5"  Part="1"
+AR Path="/52D7966D/52D79591" Ref="P6"  Part="1"
+AR Path="/52D7966B/52D79591" Ref="P7"  Part="1"
+AR Path="/52D79663/52D79591" Ref="P9"  Part="1"
+AR Path="/52D7965C/52D79591" Ref="P10"  Part="1"
+AR Path="/52D79548/52D79591" Ref="P11"  Part="1"
+F 0 "P10" V 7000 3900 50  0000 C CNN
 F 1 "CONN_4" V 7100 3900 50  0000 C CNN
 	1    7050 3900
@@
 $EndComp
 $Comp
-L ST485E U?
+L ST485E U5
 U 1 1 52D7958B
 P 4500 3900
-F 0 "U?" H 4500 3850 60  0000 C CNN
+AR Path="/52D79664/52D7958B" Ref="U5"  Part="1"
+AR Path="/52D7966E/52D7958B" Ref="U2"  Part="1"
+AR Path="/52D7966D/52D7958B" Ref="U3"  Part="1"
+AR Path="/52D7966B/52D7958B" Ref="U4"  Part="1"
+AR Path="/52D79663/52D7958B" Ref="U6"  Part="1"
+AR Path="/52D7965C/52D7958B" Ref="U7"  Part="1"
+AR Path="/52D79548/52D7958B" Ref="U8"  Part="1"
+F 0 "U7" H 4500 3850 60  0000 C CNN
 F 1 "ST485E" H 4500 3950 60  0000 C CNN
 F 2 "~" H 4550 3900 60  0000 C CNN

Commit message: Routed & ordered lux router board
Parts:
- renumbered C13 to C10, D9 to D7, F4 to F1, P8 to P5, R14 to R8, R13 to R9, U5 to U2
