File: usb_sub/usb_sub.sch (KiCad schematic (older format))
At the start: 19 parts, among them P1 CONN_1, P2 CONN_5, P3 CONN_2, U1 AURORA_CARD, U2 MICRO-B_USB, U3 FT232RL, U4 AP7333, U5 LD1117

Commit message: Mostly routed USB card
Parts:
- removed C10, C9: 1uF, symbol C
- removed C4: 100nF, symbol C
- removed P2: CONN_5, symbol CONN_5
- added D1: TX, symbol LED
- added D2: RX, symbol LED
- added D3: PWR, symbol LED
- added D4: 12V, symbol LED
- added R1, R2, R3: 270, symbol R
- added R4: 10K, symbol R
- C3: value 4.7uF -> 10uF
Connections:
- net labels removed: 5V_REG
- wire segments 83 -> 89
Other:
- moved on the sheet: C3

Commit message: Updating USB sub board
Parts:
- removed P1: CONN_1, symbol CONN_1
- removed U3: FT232RL, symbol FT232RL
- added GS?: GS3, symbol GS3
- added U?: FT232RQ, symbol FT232RQ
Connections:
- net +5V: now also GS?.3 (G3); no longer U1.13 (5V), U1.14 (5V)
- net GND: now also U?.17 (GND), U?.20 (GND), U?.24 (AGND), U?.26 (TEST), U?.33 (GND), U?.4 (GND)
- net RTS: now also U?.32 (~RTS)
- net RX: now also U?.2 (RXD)
- net TX: now also U?.30 (TXD)
- net VDD: now also GS?.1 (G1), U?.19 (VCC)
- net at U2.3 (D+): now also U?.14 (USBDP)
- net at U2.2 (D-): now also U?.15 (USBDM)
- net at C5.1, GS1.3 (G3): now also U?.16 (3v3_OUT)
- net at D2.2 (K): now also U?.21 (CBUS1)
- net at D1.2 (K): now also U?.22 (CBUS0)
- net at GS1.2 (G2): now also U?.1 (VCCIO)
- new net: GS?.2 (G2), U1.13 (5V), U1.14 (5V)
- no-connect marks 7 -> 11

Commit message: Starting re-layout of usbsub
Parts:
- gave numbers to parts that had none: 2
Connections:
- no-connect marks 11 -> 12
Changed lines of the file:
@@
 $EndComp
 $Comp
-L GND #PWR026
+L GND #PWR025
 U 1 1 52C8F653
 P 2100 3950
-F 0 "#PWR026" H 2100 3950 30  0001 C CNN
+F 0 "#PWR025" H 2100 3950 30  0001 C CNN
 F 1 "GND" H 2100 3880 30  0001 C CNN
 F 2 "" H 2100 3950 60  0001 C CNN
@@
 $EndComp
 $Comp
-L VDD #PWR027
+L VDD #PWR026
 U 1 1 52C8F63A
 P 1450 1950
-F 0 "#PWR027" H 1450 2050 30  0001 C CNN
+F 0 "#PWR026" H 1450 2050 30  0001 C CNN
 F 1 "VDD" H 1450 2060 30  0000 C CNN
 F 2 "" H 1450 1950 60  0001 C CNN
@@
 $EndComp
 $Comp
-L GND #PWR028
+L GND #PWR027
 U 1 1 52C8F2DA
 P 1450 2850
-F 0 "#PWR028" H 1450 2850 30  0001 C CNN
+F 0 "#PWR027" H 1450 2850 30  0001 C CNN
 F 1 "GND" H 1450 2780 30  0001 C CNN
 F 2 "" H 1450 2850 60  0001 C CNN
@@
 $EndComp
 $Comp
-L GS3 GS?
+L GS3 GS2
 U 1 1 53B4301E
 P 8250 1500
-F 0 "GS?" H 8300 1700 50  0000 C CNN
+F 0 "GS2" H 8300 1700 50  0000 C CNN
 F 1 "GS3" H 8300 1301 40  0000 C CNN
 F 2 "" H 8250 1500 60  0001 C CNN
@@
 	8250 2250 8250 1650
 $Comp
-L VDD #PWR?
+L VDD #PWR028
 U 1 1 53B4313A
 P 8350 1200
-F 0 "#PWR?" H 8350 1300 30  0001 C CNN
+F 0 "#PWR028" H 8350 1300 30  0001 C CNN
 F 1 "VDD" H 8350 1310 30  0000 C CNN
 F 2 "" H 8350 1200 60  0000 C CNN
@@
 	8350 1200 8350 1350
 $Comp
-L FT232RQ U?
+L FT232RQ U3
 U 1 1 53BAD3C0
 P 3100 2800
-F 0 "U?" H 3100 2950 60  0000 C CNN
+F 0 "U3" H 3100 2950 60  0000 C CNN
 F 1 "FT232RQ" H 3100 2800 60  0000 C CNN
 F 2 "" H 3100 2800 60  0000 C CNN
@@
 	1950 2600 1950 2550
 $Comp
-L GND #PWR?
+L GND #PWR029
 U 1 1 53BAD5C1
 P 3100 4150
-F 0 "#PWR?" H 3100 4150 30  0001 C CNN
+F 0 "#PWR029" H 3100 4150 30  0001 C CNN
 F 1 "GND" H 3100 4080 30  0001 C CNN
 F 2 "" H 3100 4150 60  0000 C CNN
@@
 NoConn ~ 4000 3250
 NoConn ~ 4000 3350
+NoConn ~ 1300 2650
 $EndSCHEMATC

Commit message: Debugging router
Connections:
- net +5V: now also GS2.2 (G2), U1.13 (5V), U1.14 (5V); no longer GS2.3 (G3), U5.2 (VOUT)
- new net: GS2.3 (G3), U5.2 (VOUT)
Other:
- moved on the sheet: GS2
Changed lines of the file:
@@
 	5500 2950 5400 2950
-Wire Wire Line
-	3800 6450 3800 6800
 Wire Wire Line
 	1400 3850 1400 4000
@@
 	1950 6800 2600 6800
 Wire Wire Line
-	3800 6800 3400 6800
+	3400 6800 3900 6800
 Wire Wire Line
 	2450 5800 2450 5700
@@
 L +5V #PWR06
 U 1 1 52C95643
-P 8150 1200
-F 0 "#PWR06" H 8150 1290 20  0001 C CNN
-F 1 "+5V" H 8150 1290 30  0000 C CNN
-F 2 "" H 8150 1200 60  0001 C CNN
-F 3 "" H 8150 1200 60  0001 C CNN
-	1    8150 1200
-	1    0    0    -1
+P 4000 7250
+F 0 "#PWR06" H 4000 7340 20  0001 C CNN
+F 1 "+5V" H 4000 7340 30  0000 C CNN
+F 2 "" H 4000 7250 60  0001 C CNN
+F 3 "" H 4000 7250 60  0001 C CNN
+	1    4000 7250
+	-1   0    0    1
 $EndComp
 $Comp
@@
 F 3 "" H 3000 7350 60  0001 C CNN
 	1    3000 7350
-	1    0    0    -1
-$EndComp
-$Comp
-L +5V #PWR015
-U 1 1 52C933EC
-P 3800 6450
-F 0 "#PWR015" H 3800 6540 20  0001 C CNN
-F 1 "+5V" H 3800 6540 30  0000 C CNN
-F 2 "" H 3800 6450 60  0001 C CNN
-F 3 "" H 3800 6450 60  0001 C CNN
-	1    3800 6450
 	1    0    0    -1
 $EndComp
@@
 L GS3 GS2
 U 1 1 53B4301E
-P 8250 1500
-F 0 "GS2" H 8300 1700 50  0000 C CNN
-F 1 "GS3" H 8300 1301 40  0000 C CNN
-F 2 "" H 8250 1500 60  0001 C CNN
-F 3 "" H 8250 1500 60  0001 C CNN
-	1    8250 1500
+P 4000 6950
+F 0 "GS2" H 4050 7150 50  0000 C CNN
+F 1 "GS3" H 4050 6751 40  0000 C CNN
+F 2 "" H 4000 6950 60  0001 C CNN
+F 3 "" H 4000 6950 60  0001 C CNN
+	1    4000 6950
 	0    1    1    0
 $EndComp
-Wire Wire Line
-	8150 1200 8150 1350
-Wire Wire Line
-	8250 2250 8250 1650
 $Comp
 L VDD #PWR028
 U 1 1 53B4313A
-P 8350 1200
-F 0 "#PWR028" H 8350 1300 30  0001 C CNN
-F 1 "VDD" H 8350 1310 30  0000 C CNN
-F 2 "" H 8350 1200 60  0000 C CNN
-F 3 "" H 8350 1200 60  0000 C CNN
-	1    8350 1200
-	1    0    0    -1
-$EndComp
-Wire Wire Line
-	8350 1200 8350 1350
+P 4100 6650
+F 0 "#PWR028" H 4100 6750 30  0001 C CNN
+F 1 "VDD" H 4100 6760 30  0000 C CNN
+F 2 "" H 4100 6650 60  0000 C CNN
+F 3 "" H 4100 6650 60  0000 C CNN
+	1    4100 6650
+	1    0    0    -1
+$EndComp
+Wire Wire Line
+	4100 6650 4100 6800
 $Comp
 L FT232RQ U3
@@
 $EndComp
 Wire Wire Line
-	3100 4150 3100 4100
+	3100 4100 3100 4150
 Wire Wire Line
 	2850 4100 3350 4100
@@
 NoConn ~ 4000 3350
 NoConn ~ 1300 2650
+Wire Wire Line
+	4000 7250 4000 7100
+$Comp
+L +5V #PWR?
+U 1 1 53D4111B
+P 8250 1550
+F 0 "#PWR?" H 8250 1640 20  0001 C CNN
+F 1 "+5V" H 8250 1640 30  0000 C CNN
+F 2 "" H 8250 1550 60  0001 C CNN
+F 3 "" H 8250 1550 60  0001 C CNN
+	1    8250 1550
+	1    0    0    -1
+$EndComp
+Wire Wire Line
+	8250 2250 8250 1550
 $EndSCHEMATC
